File: stepper-switch.kicad_pcb (KiCad board)
At the start: 2 copper layers, 28 x 50 mm, 27 parts, among them P1 MOLEX 70543-0004, P2 MOLEX 70543-0003, P3 MOLEX 70543-0003, P4 MOLEX 70543-0003, P5 MOLEX 70543-0003, P6 MOLEX 70543-0003, Q1 MMBF170LT1G, Q2 MMBF170LT1G

Commit message: feat: ✨ support through-hole components.
Other:
- net class Default removed
